File: documentation/PCB/Dipterv2024/Dipterv2024.kicad_sch (KiCad schematic)
At the start: 5 parts

Commit message: modell_update_hathavegleges
Parts:
- removed A? (x2): Pololu_Breakout_A4988, Module:Pololu_Breakout-16_15.2x20.3mm, symbol Driver_Motor:Pololu_Breakout_A4988
- removed U?: L7809, symbol Regulator_Linear:L7809
- removed U?: STM32F446RET6, Package_QFP:LQFP-64_10x10mm_P0.5mm, symbol MCU_ST_STM32F4:STM32F446RETx
- removed U?: AMS1117-3.3, Package_TO_SOT_SMD:SOT-223-3_TabPin2, symbol Regulator_Linear:AMS1117-3.3
- added J?: Laser modul, symbol Connector_Generic:Conn_01x02
- added J?: Gearbox, symbol Connector_Generic:Conn_01x02
- added K?: RM50-3011-85-1003, Relay_THT:Relay_SPDT_Schrack-RT1-16A-FormC_RM5mm, symbol Relay:RT314A06
- added Q?: 2N7002, Package_TO_SOT_SMD:SOT-23, symbol Transistor_FET:2N7002
- added U: SZBK07, symbol New_Library:SZBK07
- added U?: RPI 4B, Package_DFN_QFN:QFN-56-1EP_7x7mm_P0.4mm_EP3.2x3.2mm, symbol MCU_RaspberryPi:RP2040
- added U?: Waveshare stepper hat, symbol New_Library:Stepper_HAT
Connections:
- new net: Q?.1 (G), U?.5 (GPIO3)
- new net: K?.A2, Q?.3 (D)
- new net: U?.1 (IOVDD), U?.10 (IOVDD), U?.22 (IOVDD), U?.33 (IOVDD), U?.42 (IOVDD), U?.49 (IOVDD)
- new net: U?.23 (DVDD), U?.50 (DVDD)
- new net: J?.1 (Pin_1), U?.32 (GPIO21)
- new net: J?.1 (Pin_1), K?.12
- new net +12V: U.1 (VIN+)
- new net +3.3V: K?.A1
- new net +7.4V: K?.11, U.3 (+VDC)
- new net A1A2B1B2 dir: U?.1 (A1A2B1B2_dir), U?.16 (GPIO13)
- new net A1A2B1B2 enable: U?.15 (GPIO12), U?.3 (A1A2B1B2_enable)
- new net A1A2B1B2 step: U?.2 (A1A2B1B2_step), U?.30 (GPIO19)
- new net A3A4B3B4 dir: U?.36 (GPIO24), U?.4 (A3A4B3B4_dir)
- new net A3A4B3B4 enable: U?.6 (A3A4B3B4_enable), U?.6 (GPIO4)
- new net A3A4B3B4 step: U?.29 (GPIO18), U?.5 (A3A4B3B4_step)
- new net GND: J?.2 (Pin_2), Q?.2 (S)
- new net GND2: J?.2 (Pin_2), U.2 (VIN-), U.4 (-VDC)

Commit message: update
Parts:
- added U5, U6: ES011, symbol New_Library:ES011
- gave numbers to parts that had none: 6
- renumbered U to U3
Connections:
- net +3.3V: now also U5.1 (VCC)
- net GND: now also U1.57 (GND), U6.3 (GND)
- net at U1.5 (GPIO3): no longer Q1.1 (G)
- net Vegallas2 VCC: now reaches U1.14 (GPIO11)
- net Vegallas2 VCC: now also U6.1 (VCC)
- net Vegallas2 SIG: now reaches U1.2 (GPIO0)
- net Vegallas2 SIG: now also U6.2 (OUT)
- net Weapon enable: now reaches U1.31 (GPIO20)
- net Weapon enable: now also Q1.1 (G)
- net Laser enable: now reaches U1.32 (GPIO21), U4.1 (Pin_1)
- net Vegallas1 GND: now reaches U1.34 (GPIO22)
- net Vegallas1 GND: now also U5.3 (GND)
- net Vegallas1 SIG: now reaches U1.39 (GPIO27_ADC1)
- net Vegallas1 SIG: now also U5.2 (OUT)
- no-connect marks 0 -> 39
Other:
- moved on the sheet: J1, K1, Q1, U1, U2, U3, U4
